Commit message: Started task 3 grasping
Co-authored-by: Giulio Mazzaroppi <Giulio-Mazzar@users.noreply.github.com>
Co-authored-by: giacomo2k2 <giacomo2k2@users.noreply.github.com>

File: src/pal_gripper/pal_gripper_description/urdf/gripper.gazebo.xacro (robot description, xacro)
@@ -15,11 +15,11 @@
   <xacro:macro name="finger_gazebo" params="name">
     <gazebo reference="${name}_link">
-      <kp>1000000.0</kp>
-      <kd>1.0</kd>
-      <mu1>1.0</mu1>
-      <mu2>1.0</mu2>
+      <kp>100000.0</kp>
+      <kd>10.0</kd>
+      <mu1>10000.0</mu1>
+      <mu2>10000.0</mu2>
       <fdir1>0 0 0</fdir1>
       <maxVel>1.0</maxVel>
-      <minDepth>0.1</minDepth>
+      <minDepth>0.001</minDepth>
       <material>Gazebo/Black</material>
     </gazebo>
@@ -30,2 +30,3 @@
   </xacro:macro>
 </robot>
+<!-- mu1 10, mu2 10, minDepth 0.1, kp 1000000, kd 1 -->

File: src/pal_gripper/pal_gripper_description/urdf/gripper.urdf.xacro (robot description, xacro)
@@ -84,5 +84,5 @@
     <limit effort="16" lower="0.0" upper="0.045" velocity="0.05" />
     <calibration rising="0.0" />
-    <dynamics damping="80" friction="2.0"/>
+    <dynamics damping="80" friction="10.0"/>
     <safety_controller k_position="20"
                        k_velocity="20"
@@ -122,5 +122,5 @@
     <limit effort="16" lower="0" upper="0.045" velocity="0.05" />
     <calibration rising="0.0" />
-    <dynamics damping="80" friction="2.0"/>
+    <dynamics damping="80" friction="10.0"/>
     <safety_controller k_position="20"
                        k_velocity="20"

Commit message: Tried to grasp unsuccessfully
Co-authored-by: giacomo2k2 <giacomo2k2@users.noreply.github.com>
Co-authored-by: Giulio Mazzaroppi <Giulio-Mazzar@users.noreply.github.com>

File: src/pal_gripper/pal_gripper_description/urdf/gripper.gazebo.xacro (robot description, xacro)
@@ -13,4 +13,5 @@
  -->
 <robot xmlns:xacro="http://ros.org/wiki/xacro">
+  <!--
   <xacro:macro name="finger_gazebo" params="name">
     <gazebo reference="${name}_link">
@@ -29,4 +30,25 @@
     </gazebo>
   </xacro:macro>
+  -->
+  <!-- <xacro:macro name="finger_gazebo" params="name">
+    <gazebo reference="${name}_link">
+      <kp>1000000.0</kp>
+      <kd>1.0</kd>
+      <mu1>200.0</mu1>
+      <mu2>200.0</mu2>
+      <maxVel>0.0</maxVel>
+      <minDepth>0.001</minDepth>
+      <material>Gazebo/Black</material>
+    </gazebo>
+  </xacro:macro> -->
+  <xacro:macro name="finger_gazebo" params="name">
+    <gazebo reference="${name}_link">
+      <kp>100000.0</kp>
+      <kd>100.0</kd>
+      <mu1>Inf</mu1>  <mu2>Inf</mu2>
+      <minDepth>0.0</minDepth>
+      <maxVel>0.01</maxVel>
+    </gazebo>
+  </xacro:macro>
 </robot>
 <!-- mu1 10, mu2 10, minDepth 0.1, kp 1000000, kd 1 -->

File: src/pal_gripper/pal_gripper_description/urdf/gripper.urdf.xacro (robot description, xacro)
@@ -67,6 +67,12 @@
       <material name="Black"/>
     </visual>
+    <!-- <collision>
+      <origin rpy="0 0 3.1415" xyz="0.005 0 -0.165" />
+      <geometry>
+        <box size="0.01 0.05 0.11"/>
+      </geometry>
+    </collision> -->
     <collision>
-      <origin rpy="0 0 3.1415" xyz="0.005 0 -0.165" />
+      <origin rpy="0 0 3.1415" xyz="0.005 0 -0.12" />
       <geometry>
         <box size="0.01 0.05 0.11"/>
@@ -84,5 +90,5 @@
     <limit effort="16" lower="0.0" upper="0.045" velocity="0.05" />
     <calibration rising="0.0" />
-    <dynamics damping="80" friction="10.0"/>
+    <dynamics damping="1.0" friction="1.0"/>
     <safety_controller k_position="20"
                        k_velocity="20"
@@ -105,6 +111,12 @@
       <material name="Black"/>
     </visual>
+    <!-- <collision>
+      <origin rpy="0 0 3.1415" xyz="-0.005 0 -0.165" />
+      <geometry>
+        <box size="0.01 0.05 0.11"/>
+      </geometry>
+    </collision> -->
     <collision>
-      <origin rpy="0 0 3.1415" xyz="-0.005 0 -0.165" />
+      <origin rpy="0 0 3.1415" xyz="-0.005 0 -0.12" />
       <geometry>
         <box size="0.01 0.05 0.11"/>
@@ -122,5 +134,5 @@
     <limit effort="16" lower="0" upper="0.045" velocity="0.05" />
     <calibration rising="0.0" />
-    <dynamics damping="80" friction="10.0"/>
+    <dynamics damping="1.0" friction="1.0"/>
     <safety_controller k_position="20"
                        k_velocity="20"

Commit message: Tutto tuo frasco duda, day nr. 2 of working over friction for the gazebo engine for grasping achieving without ifra link attacher.
Co-authored-by: giacomo2k2 <giacomo2k2@users.noreply.github.com>

File: src/pal_gripper/pal_gripper_description/urdf/gripper.gazebo.xacro (robot description, xacro)
@@ -42,11 +42,13 @@
     </gazebo>
   </xacro:macro> -->
-  <xacro:macro name="finger_gazebo" params="name">
+ <xacro:macro name="finger_gazebo" params="name">
     <gazebo reference="${name}_link">
       <kp>100000.0</kp>
       <kd>10.0</kd>
-      <mu1>1000</mu1>  <mu2>1000</mu2>
-      <minDepth>0.0</minDepth>
-      <maxVel>0.01</maxVel>
+      <mu1>1.0</mu1>
+      <mu2>1.0</mu2>
+      <minDepth>0.001</minDepth>
+      <maxVel>0.0</maxVel>
+      <material>Gazebo/Black</material>
     </gazebo>
   </xacro:macro>

File: src/pal_gripper/pal_gripper_description/urdf/gripper.urdf.xacro (robot description, xacro)
@@ -67,14 +67,8 @@
       <material name="Black"/>
     </visual>
-    <!-- <collision>
-      <origin rpy="0 0 3.1415" xyz="0.005 0 -0.165" />
+    <collision>
+      <origin rpy="0 0 3.1415" xyz="0.005 0 -0.1425" />
       <geometry>
-        <box size="0.01 0.05 0.11"/>
-      </geometry>
-    </collision> -->
-    <collision>
-      <origin rpy="0 0 3.1415" xyz="0.005 0 -0.12" />
-      <geometry>
-        <box size="0.01 0.05 0.11"/>
+        <box size="0.01 0.05 0.155"/>
       </geometry>
     </collision>
@@ -88,12 +82,8 @@
     <child link="${name}_right_finger_link" />
     <axis xyz="1 0 0" />
-    <limit effort="16" lower="0.0" upper="0.045" velocity="0.05" />
+    <limit effort="1000.0" lower="0.0" upper="0.045" velocity="0.5" />
     <calibration rising="0.0" />
-    <dynamics damping="1.0" friction="1.0"/>
-    <safety_controller k_position="20"
-                       k_velocity="20"
-                       soft_lower_limit="${0.0 + gripper_eps}"
-                       soft_upper_limit="${0.045 - gripper_eps}" />
-  </joint>
+    <dynamics damping="0.0" friction="0.0"/>
+    </joint>
   <link name="${name}_left_finger_link">
     <inertial>
@@ -111,14 +101,8 @@
       <material name="Black"/>
     </visual>
-    <!-- <collision>
-      <origin rpy="0 0 3.1415" xyz="-0.005 0 -0.165" />
+    <collision>
+      <origin rpy="0 0 3.1415" xyz="-0.005 0 -0.1425" />
       <geometry>
-        <box size="0.01 0.05 0.11"/>
-      </geometry>
-    </collision> -->
-    <collision>
-      <origin rpy="0 0 3.1415" xyz="-0.005 0 -0.12" />
-      <geometry>
-        <box size="0.01 0.05 0.11"/>
+        <box size="0.01 0.05 0.155"/>
       </geometry>
     </collision>
@@ -132,12 +116,8 @@
     <child link="${name}_left_finger_link" />
     <axis xyz="-1 0 0" />
-    <limit effort="16" lower="0" upper="0.045" velocity="0.05" />
+    <limit effort="50.0" lower="0" upper="0.045" velocity="0.5" />
     <calibration rising="0.0" />
-    <dynamics damping="1.0" friction="1.0"/>
-    <safety_controller k_position="20"
-                       k_velocity="20"
-                       soft_lower_limit="${0.0 + gripper_eps}"
-                       soft_upper_limit="${0.045 - gripper_eps}" />
-  </joint>
+    <dynamics damping="1.0" friction="0.0"/>
+    </joint>
   <!-- Grasping frame -->
   <joint name="${name}_grasping_frame_joint" type="fixed">
@@ -158,11 +138,11 @@
   <xacro:finger_gazebo name="${name}_right_finger"/>
   <gazebo reference="${name}_link">
-      <gravity>0</gravity>
+      <gravity>1</gravity>
   </gazebo>
   <gazebo reference="${name}_left_finger">
-      <gravity>0</gravity>
+      <gravity>1</gravity>
   </gazebo>
   <gazebo reference="${name}_right_finger">
-      <gravity>0</gravity>
+      <gravity>1</gravity>
   </gazebo>
  </xacro:macro>

File: src/tiago_robot/tiago_description/robots/tiago.urdf.xacro (robot description, xacro)
@@ -137,3 +137,20 @@
       </inertial>
   </link>
+  <gazebo>
+    <plugin name="gazebo_grasp_fix" filename="libgazebo_grasp_fix.so">
+      <arm>
+        <arm_name>tiago_arm</arm_name>
+        <palm_link>gripper_link</palm_link>
+        <gripper_link>gripper_left_finger_link</gripper_link>
+        <gripper_link>gripper_right_finger_link</gripper_link>
+      </arm>
+      <forces_angle_tolerance>100</forces_angle_tolerance>
+      <update_rate>20</update_rate>
+      <grip_count_threshold>4</grip_count_threshold>
+      <max_grip_count>10</max_grip_count>
+      <release_tolerance>0.005</release_tolerance>
+      <disable_collisions_on_attach>false</disable_collisions_on_attach>
+      <contact_topic>physics/contacts</contact_topic>
+    </plugin>
+  </gazebo>
 </robot>
